File: pcb/skibidi-usb-c-hub.kicad_pcb (KiCad board)
At the start: 2 copper layers, 0 parts

Commit message: pcb half way done
Parts:
- added C1: 100n, Capacitor_SMD:C_0402_1005Metric, F.Cu at (35.8, 51.4)
- added C2: 100n, Capacitor_SMD:C_0402_1005Metric, F.Cu at (35.8, 53.4)
- added D1: 5V, Diode_SMD:D_SOD-523, F.Cu at (132.8, 78.1)
- added F1: 2A, Fuse:Fuse_1206_3216Metric, F.Cu at (133.8, 72.3)
- added FB1: 220Ω@100MHz, Resistor_SMD:R_0805_2012Metric_Pad1.20x1.40mm_HandSolder, F.Cu at (133.4, 75.4)
- added R1: 56k, Resistor_SMD:R_0603_1608Metric, F.Cu at (112.8, 98.5)
- added R2: 56k, Resistor_SMD:R_0603_1608Metric, F.Cu at (112.8, 101.0)
- added R3: 56k, Resistor_SMD:R_0603_1608Metric, F.Cu at (129.4, 104.7)
- added R4: 56k, Resistor_SMD:R_0603_1608Metric, F.Cu at (129.4, 107.2)
- added R5: 56k, Resistor_SMD:R_0603_1608Metric, F.Cu at (142.3, 104.7)
- added R6: 56k, Resistor_SMD:R_0603_1608Metric, F.Cu at (142.3, 107.2)
- added R7: 56k, Resistor_SMD:R_0603_1608Metric, F.Cu at (140.6, 80.9)
- added R8: 56k, Resistor_SMD:R_0603_1608Metric, F.Cu at (140.6, 83.4)
- added TP1: TestPoint, TestPoint:TestPoint_Pad_D1.0mm, F.Cu at (132.5, 80.9)
- added U1: CH334P, easyeda2kicad:QFN-16_L3.0-W3.0-P0.50-BL-EP1.7, F.Cu at (38.4, 52.6)
- added USB1: AM90, easyeda2kicad:USB-AM-TH_AM90, F.Cu at (38.8, 34.0)
- added USB2: TYPE-C 16PIN 2MD(073), easyeda2kicad:USB-C-SMD_TYPE-C-6PIN-2MD-073, F.Cu at (43.7, 42.9)
- added USB3: TYPE-C 16PIN 2MD(073), easyeda2kicad:USB-C-SMD_TYPE-C-6PIN-2MD-073, F.Cu at (43.7, 62.9)
- added USB4: TYPE-C 16PIN 2MD(073), easyeda2kicad:USB-C-SMD_TYPE-C-6PIN-2MD-073, F.Cu at (33.8, 62.9)
- added USB5: TYPE-C 16PIN 2MD(073), easyeda2kicad:USB-C-SMD_TYPE-C-6PIN-2MD-073, F.Cu at (33.8, 42.9)
Routing:
- net /USB A Upstream/D-: track 0.00 -> 27.8 mm, vias 0 -> 1
- net /USB A Upstream/D+: track 0.00 -> 26.5 mm, vias 0 -> 1
- net /USB C 4/D+: track 0.00 -> 23.3 mm
- net /USB C 4/D-: track 0.00 -> 22.6 mm
- net /USB C 2/D-: track 0.00 -> 17.9 mm
- net /USB C 2/D+: track 0.00 -> 17.9 mm
- net /USB C 3/D+: track 0.00 -> 17.4 mm
- net /USB C 3/D-: track 0.00 -> 16.1 mm
- net /USB C 1/D+: track 0.00 -> 12.3 mm
- net /USB C 1/D-: track 0.00 -> 11.7 mm
- net (no net): vias 0 -> 4
Other:
- board outline added: 17.5 x 39 mm
