File: pcb/skibidi-usb-c-hub.kicad_sch (KiCad schematic)
At the start: 0 parts

Commit message: schematic done
Parts:
- added C1, C2: 100n, Capacitor_SMD:C_0402_1005Metric, symbol Device:C
- added U1: CH334P, easyeda2kicad:QFN-16_L3.0-W3.0-P0.50-BL-EP1.7, symbol easyeda2kicad:CH334P
Connections:
- new net +3V3: C2.1, U1.16 (VDD33)
- new net GND: C1.2, C2.2, U1.17 (GND)
- new net USB A Upstream/D+: U1.12 (DPU)
- new net USB A Upstream/D-: U1.11 (DMU)
- new net USB C 1/D+: U1.10 (DP1)
- new net USB C 1/D-: U1.9 (DM1)
- new net USB C 2/D+: U1.8 (DP2)
- new net USB C 2/D-: U1.7 (DM2)
- new net USB C 3/D+: U1.6 (DP3)
- new net USB C 3/D-: U1.5 (DM3)
- new net USB C 4/D+: U1.4 (DP4)
- new net USB C 4/D-: U1.3 (DM4)
- new net VBUS: C1.1, U1.15 (V5)
Other:
- added sheet USB A Upstream (usb_a.kicad_sch)
- added sheet USB C 1 (usb_c.kicad_sch)
- added sheet USB C 2 (usb_c.kicad_sch)
- added sheet USB C 3 (usb_c.kicad_sch)
- added sheet USB C 4 (usb_c.kicad_sch)

Commit message: finished pcb and bom, added schematic pdf, step file for pcb, and gerbers
Parts:
- added C9: 220u, Capacitor_SMD:CP_Elec_6.3x5.8, symbol Device:C_Polarized
- C2: value 100n -> 4.7u; LCSC Part # C1525 -> C23733
Connections:
- net GND: now also C9.2
- net VBUS: now also C9.1
Changed lines of the file:
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@@
 	(generator_version "9.0")
 	(paper "A4")
+	(junction
+		(at 139.7 53.34)
+		(diameter 0)
+		(color 0 0 0 0)
+	)
+	(junction
+		(at 139.7 60.96)
+		(diameter 0)
+		(color 0 0 0 0)
+	)
 	(wire
 		(pts
@@
 	(wire
 		(pts
+			(xy 127 60.96) (xy 139.7 60.96)
+		)
+		(stroke
+			(width 0)
+			(type default)
+		)
+	)
+	(wire
+		(pts
 			(xy 170.18 87.63) (xy 177.8 87.63)
 		)
@@
 		(pts
 			(xy 135.89 86.36) (xy 138.43 86.36)
+		)
+		(stroke
+			(width 0)
+			(type default)
+		)
+	)
+	(wire
+		(pts
+			(xy 127 53.34) (xy 139.7 53.34)
 		)
 		(stroke
@@
 			)
 		)
-		(property "Value" "100n"
+		(property "Value" "4.7u"
 			(at 156.21 59.0549 0)
 			(effects
@@
 			)
 		)
-		(property "LCSC Part #" "C1525"
+		(property "LCSC Part #" "C23733"
 			(at 152.4 57.15 0)
 			(effects
@@
 					(unit 1)
 				)
+			)
+		)
+	)
+	(symbol
+		(lib_id "Device:C_Polarized")
+		(at 127 57.15 0)
+		(unit 1)
+		(exclude_from_sim no)
+		(in_bom yes)
+		(on_board yes)
+		(dnp no)
+		(property "Reference" "C9"
+			(at 130.81 55.372 0)
+			(effects
+				(font
+					(size 1.27 1.27)
+				)
+				(justify left)
+			)
+		)
+		(property "Value" "220u"
+			(at 130.81 59.182 0)
+			(effects
+				(font
+					(size 1.27 1.27)
+				)
+				(justify left)
+			)
+		)
+		(property "Footprint" "Capacitor_SMD:CP_Elec_6.3x5.8"
+			(at 127.9652 60.96 0)
+			(effects
+				(font
+					(size 1.27 1.27)
+				)
+				(hide yes)
+			)
+		)
+		(property "Datasheet" "~"
+			(at 127 57.15 0)
+			(effects
+				(font
+					(size 1.27 1.27)
+				)
+				(hide yes)
+			)
+		)
+		(property "Description" "Polarized capacitor"
+			(at 127 57.15 0)
+			(effects
+				(font
+					(size 1.27 1.27)
+				)
+				(hide yes)
+			)
+		)
+		(property "LCSC Part #" "C5246513"
+			(at 127 57.15 0)
+			(effects
+				(font
+					(size 1.27 1.27)
+				)
+				(hide yes)
+			)
+		)
+		(pin "2"
+		)
+		(pin "1"
+		)
+		(instances
+			(project ""
+				(path "/ba8238db-cbbe-49a0-8684-36588779fc6b"
+					(reference "C9")
+					(unit 1)
+				)
