File: pcb/usb_a.kicad_sch (KiCad schematic)
At the start: 5 parts

Commit message: pcb half way done
Parts:
- gave numbers to parts that had none: 4
Changed lines of the file:
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@@
 		(dnp no)
 		(fields_autoplaced yes)
-		(property "Reference" "F?"
+		(property "Reference" "F1"
 			(at 156.21 87.63 90)
 			(effects
@@
 			(project "skibidi-usb-c-hub"
 				(path "/ba8238db-cbbe-49a0-8684-36588779fc6b/d55cf89a-dfdd-4a58-8a8b-d23172701bd8"
-					(reference "F?")
+					(reference "F1")
 					(unit 1)
 				)
@@
 		(on_board yes)
 		(dnp no)
-		(property "Reference" "TP?"
+		(property "Reference" "TP1"
 			(at 195.326 88.392 0)
 			(effects
@@
 			(project "skibidi-usb-c-hub"
 				(path "/ba8238db-cbbe-49a0-8684-36588779fc6b/d55cf89a-dfdd-4a58-8a8b-d23172701bd8"
-					(reference "TP?")
+					(reference "TP1")
 					(unit 1)
 				)
@@
 		(on_board yes)
 		(dnp no)
-		(property "Reference" "D?"
+		(property "Reference" "D1"
 			(at 170.688 101.092 90)
 			(effects
@@
 			(project "skibidi-usb-c-hub"
 				(path "/ba8238db-cbbe-49a0-8684-36588779fc6b/d55cf89a-dfdd-4a58-8a8b-d23172701bd8"
-					(reference "D?")
+					(reference "D1")
 					(unit 1)
 				)
@@
 		(dnp no)
 		(fields_autoplaced yes)
-		(property "Reference" "#PWR02"
+		(property "Reference" "#PWR010"
 			(at 139.7 120.65 0)
 			(effects
@@
 			(project ""
 				(path "/ba8238db-cbbe-49a0-8684-36588779fc6b/d55cf89a-dfdd-4a58-8a8b-d23172701bd8"
-					(reference "#PWR02")
+					(reference "#PWR010")
 					(unit 1)
 				)
@@
 		(dnp no)
 		(fields_autoplaced yes)
-		(property "Reference" "#PWR?"
+		(property "Reference" "#PWR08"
 			(at 191.77 100.33 0)
 			(effects
@@
 			(project "skibidi-usb-c-hub"
 				(path "/ba8238db-cbbe-49a0-8684-36588779fc6b/d55cf89a-dfdd-4a58-8a8b-d23172701bd8"
-					(reference "#PWR?")
+					(reference "#PWR08")
 					(unit 1)
 				)
@@
 		(dnp no)
 		(fields_autoplaced yes)
-		(property "Reference" "#PWR?"
+		(property "Reference" "#PWR09"
 			(at 167.64 115.57 0)
 			(effects
@@
 			(project "skibidi-usb-c-hub"
 				(path "/ba8238db-cbbe-49a0-8684-36588779fc6b/d55cf89a-dfdd-4a58-8a8b-d23172701bd8"
-					(reference "#PWR?")
+					(reference "#PWR09")
 					(unit 1)
 				)
@@
 		(dnp no)
 		(fields_autoplaced yes)
-		(property "Reference" "FB?"
+		(property "Reference" "FB1"
 			(at 179.0192 87.63 90)
 			(effects
@@
 			(project "skibidi-usb-c-hub"
 				(path "/ba8238db-cbbe-49a0-8684-36588779fc6b/d55cf89a-dfdd-4a58-8a8b-d23172701bd8"
-					(reference "FB?")
-					(unit 1)
-				)
+					(reference "FB1")
+					(unit 1)
+				)

Commit message: finished pcb and bom, added schematic pdf, step file for pcb, and gerbers
Parts:
- TP1: footprint TestPoint:TestPoint_Pad_D1.0mm -> TestPoint:TestPoint_Pad_D2.5mm
Changed lines of the file:
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@@
 			)
 		)
-		(property "Footprint" "TestPoint:TestPoint_Pad_D1.0mm"
+		(property "Footprint" "TestPoint:TestPoint_Pad_D2.5mm"
 			(at 201.93 93.98 0)
 			(effects
