File: pcb/usb_c.kicad_sch (KiCad schematic)
At the start: 3 parts

Commit message: pcb half way done
Parts:
- renumbered R6 to R1, R1 to R2
Changed lines of the file:
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@@
 		(dnp no)
 		(fields_autoplaced yes)
-		(property "Reference" "#PWR03"
+		(property "Reference" "#PWR011"
 			(at 139.7 91.44 0)
 			(effects
@@
 			(project "skibidi-usb-c-hub"
 				(path "/ba8238db-cbbe-49a0-8684-36588779fc6b/6f59b006-c39b-4f95-9bd5-f3ad5c9f2e1d"
-					(reference "#PWR012")
+					(reference "#PWR020")
 					(unit 1)
 				)
 				(path "/ba8238db-cbbe-49a0-8684-36588779fc6b/a20e208f-9c1f-498b-b7e6-c187e8f066dd"
-					(reference "#PWR03")
+					(reference "#PWR011")
 					(unit 1)
 				)
 				(path "/ba8238db-cbbe-49a0-8684-36588779fc6b/a3f216c1-5ccc-45d3-8b9e-12c0f2e53f02"
-					(reference "#PWR06")
+					(reference "#PWR014")
 					(unit 1)
 				)
 				(path "/ba8238db-cbbe-49a0-8684-36588779fc6b/fb8800a7-8efe-42d7-a8d1-e327d54fdf66"
-					(reference "#PWR09")
+					(reference "#PWR017")
 					(unit 1)
 				)
@@
 		(dnp no)
 		(fields_autoplaced yes)
-		(property "Reference" "#PWR04"
+		(property "Reference" "#PWR013"
 			(at 139.7 124.46 0)
 			(effects
@@
 			(project "skibidi-usb-c-hub"
 				(path "/ba8238db-cbbe-49a0-8684-36588779fc6b/6f59b006-c39b-4f95-9bd5-f3ad5c9f2e1d"
-					(reference "#PWR014")
+					(reference "#PWR022")
 					(unit 1)
 				)
 				(path "/ba8238db-cbbe-49a0-8684-36588779fc6b/a20e208f-9c1f-498b-b7e6-c187e8f066dd"
-					(reference "#PWR04")
+					(reference "#PWR013")
 					(unit 1)
 				)
 				(path "/ba8238db-cbbe-49a0-8684-36588779fc6b/a3f216c1-5ccc-45d3-8b9e-12c0f2e53f02"
-					(reference "#PWR08")
+					(reference "#PWR016")
 					(unit 1)
 				)
 				(path "/ba8238db-cbbe-49a0-8684-36588779fc6b/fb8800a7-8efe-42d7-a8d1-e327d54fdf66"
-					(reference "#PWR011")
+					(reference "#PWR019")
 					(unit 1)
 				)
@@
 		(dnp no)
 		(fields_autoplaced yes)
-		(property "Reference" "#PWR05"
+		(property "Reference" "#PWR012"
 			(at 101.6 104.14 0)
 			(effects
@@
 			(project "skibidi-usb-c-hub"
 				(path "/ba8238db-cbbe-49a0-8684-36588779fc6b/6f59b006-c39b-4f95-9bd5-f3ad5c9f2e1d"
-					(reference "#PWR013")
+					(reference "#PWR021")
 					(unit 1)
 				)
 				(path "/ba8238db-cbbe-49a0-8684-36588779fc6b/a20e208f-9c1f-498b-b7e6-c187e8f066dd"
-					(reference "#PWR05")
+					(reference "#PWR012")
 					(unit 1)
 				)
 				(path "/ba8238db-cbbe-49a0-8684-36588779fc6b/a3f216c1-5ccc-45d3-8b9e-12c0f2e53f02"
-					(reference "#PWR07")
+					(reference "#PWR015")
 					(unit 1)
 				)
 				(path "/ba8238db-cbbe-49a0-8684-36588779fc6b/fb8800a7-8efe-42d7-a8d1-e327d54fdf66"
-					(reference "#PWR010")
+					(reference "#PWR018")
 					(unit 1)
 				)
@@
 		(dnp no)
 		(fields_autoplaced yes)
-		(property "Reference" "R1"
+		(property "Reference" "R2"
 			(at 107.95 97.79 90)
 			(effects
@@
 			(project "skibidi-usb-c-hub"
 				(path "/ba8238db-cbbe-49a0-8684-36588779fc6b/6f59b006-c39b-4f95-9bd5-f3ad5c9f2e1d"
-					(reference "R7")
+					(reference "R8")
 					(unit 1)
 				)
 				(path "/ba8238db-cbbe-49a0-8684-36588779fc6b/a20e208f-9c1f-498b-b7e6-c187e8f066dd"
-					(reference "R1")
+					(reference "R2")
 					(unit 1)
 				)
 				(path "/ba8238db-cbbe-49a0-8684-36588779fc6b/a3f216c1-5ccc-45d3-8b9e-12c0f2e53f02"
-					(reference "R3")
+					(reference "R4")
 					(unit 1)
 				)
 				(path "/ba8238db-cbbe-49a0-8684-36588779fc6b/fb8800a7-8efe-42d7-a8d1-e327d54fdf66"
-					(reference "R5")
+					(reference "R6")
 					(unit 1)
 				)
@@
 		(dnp no)
 		(fields_autoplaced yes)
-		(property "Reference" "R?"
+		(property "Reference" "R1"
 			(at 115.57 95.25 90)
 			(effects
@@
 			(project "skibidi-usb-c-hub"
 				(path "/ba8238db-cbbe-49a0-8684-36588779fc6b/6f59b006-c39b-4f95-9bd5-f3ad5c9f2e1d"
-					(reference "R6")
+					(reference "R7")
 					(unit 1)
 				)
 				(path "/ba8238db-cbbe-49a0-8684-36588779fc6b/a20e208f-9c1f-498b-b7e6-c187e8f066dd"
-					(reference "R?")
+					(reference "R1")
 					(unit 1)
 				)
 				(path "/ba8238db-cbbe-49a0-8684-36588779fc6b/a3f216c1-5ccc-45d3-8b9e-12c0f2e53f02"
-					(reference "R2")
+					(reference "R3")
 					(unit 1)
 				)
 				(path "/ba8238db-cbbe-49a0-8684-36588779fc6b/fb8800a7-8efe-42d7-a8d1-e327d54fdf66"
-					(reference "R4")
-					(unit 1)
-				)
+					(reference "R5")
+					(unit 1)
+				)

Commit message: finished pcb and bom, added schematic pdf, step file for pcb, and gerbers
Parts:
- added C5: 10u, Capacitor_SMD:C_0603_1608Metric, symbol Device:C
Connections:
- net GND: now also C5.2
- net VBUS: now also C5.1
Changed lines of the file:
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@@
+	)
+	(symbol
+		(lib_id "Device:C")
+		(at 165.1 82.55 0)
+		(unit 1)
+		(exclude_from_sim no)
+		(in_bom yes)
+		(on_board yes)
+		(dnp no)
+		(property "Reference" "C5"
+			(at 168.91 80.6449 0)
+			(effects
+				(font
+					(size 1.27 1.27)
+				)
+				(justify left)
+			)
+		)
+		(property "Value" "10u"
+			(at 168.91 84.4549 0)
+			(effects
+				(font
+					(size 1.27 1.27)
+				)
+				(justify left)
+			)
+		)
+		(property "Footprint" "Capacitor_SMD:C_0603_1608Metric"
+			(at 166.0652 86.36 0)
+			(effects
+				(font
+					(size 1.27 1.27)
+				)
+				(hide yes)
+			)
+		)
+		(property "Datasheet" "~"
+			(at 165.1 82.55 0)
+			(effects
+				(font
+					(size 1.27 1.27)
+				)
+				(hide yes)
+			)
+		)
+		(property "Description" "Unpolarized capacitor"
+			(at 165.1 82.55 0)
+			(effects
+				(font
+					(size 1.27 1.27)
+				)
+				(hide yes)
+			)
+		)
+		(property "LCSC Part #" "C96446"
+			(at 165.1 82.55 0)
+			(effects
+				(font
+					(size 1.27 1.27)
+				)
+				(hide yes)
+			)
+		)
+		(pin "2"
+		)
+		(pin "1"
+		)
+		(instances
+			(project "skibidi-usb-c-hub"
+				(path "/ba8238db-cbbe-49a0-8684-36588779fc6b/6f59b006-c39b-4f95-9bd5-f3ad5c9f2e1d"
+					(reference "C8")
+					(unit 1)
+				)
+				(path "/ba8238db-cbbe-49a0-8684-36588779fc6b/a20e208f-9c1f-498b-b7e6-c187e8f066dd"
+					(reference "C5")
+					(unit 1)
+				)
+				(path "/ba8238db-cbbe-49a0-8684-36588779fc6b/a3f216c1-5ccc-45d3-8b9e-12c0f2e53f02"
+					(reference "C6")
+					(unit 1)
+				)
+				(path "/ba8238db-cbbe-49a0-8684-36588779fc6b/fb8800a7-8efe-42d7-a8d1-e327d54fdf66"
+					(reference "C7")
+					(unit 1)
+				)
+			)
+		)
 	)
 	(symbol
@@
 	)
 	(symbol
+		(lib_id "power:GND")
+		(at 165.1 86.36 0)
+		(unit 1)
+		(exclude_from_sim no)
+		(in_bom yes)
+		(on_board yes)
+		(dnp no)
+		(fields_autoplaced yes)
+		(property "Reference" "#PWR024"
+			(at 165.1 92.71 0)
+			(effects
+				(font
+					(size 1.27 1.27)
+				)
+				(hide yes)
+			)
+		)
+		(property "Value" "GND"
+			(at 165.1 91.44 0)
+			(effects
+				(font
+					(size 1.27 1.27)
+				)
+				(hide yes)
+			)
+		)
+		(property "Footprint" ""
+			(at 165.1 86.36 0)
+			(effects
+				(font
+					(size 1.27 1.27)
+				)
+				(hide yes)
+			)
+		)
+		(property "Datasheet" ""
+			(at 165.1 86.36 0)
+			(effects
+				(font
+					(size 1.27 1.27)
+				)
+				(hide yes)
+			)
+		)
+		(property "Description" "Power symbol creates a global label with name \"GND\" , ground"
+			(at 165.1 86.36 0)
+			(effects
+				(font
+					(size 1.27 1.27)
+				)
+				(hide yes)
+			)
+		)
+		(pin "1"
+		)
+		(instances
+			(project "skibidi-usb-c-hub"
+				(path "/ba8238db-cbbe-49a0-8684-36588779fc6b/6f59b006-c39b-4f95-9bd5-f3ad5c9f2e1d"
+					(reference "#PWR027")
+					(unit 1)
+				)
+				(path "/ba8238db-cbbe-49a0-8684-36588779fc6b/a20e208f-9c1f-498b-b7e6-c187e8f066dd"
+					(reference "#PWR024")
+					(unit 1)
+				)
+				(path "/ba8238db-cbbe-49a0-8684-36588779fc6b/a3f216c1-5ccc-45d3-8b9e-12c0f2e53f02"
+					(reference "#PWR025")
+					(unit 1)
+				)
+				(path "/ba8238db-cbbe-49a0-8684-36588779fc6b/fb8800a7-8efe-42d7-a8d1-e327d54fdf66"
+					(reference "#PWR026")
+					(unit 1)
+				)
+			)
+		)
+	)
+	(symbol
 		(lib_id "easyeda2kicad:TYPE-C16PIN2MD(073)")
 		(at 139.7 101.6 0)
@@
 					(unit 1)
 				)
+			)
+		)
+	)
+	(symbol
+		(lib_id "power:VBUS")
+		(at 165.1 78.74 0)
+		(unit 1)
+		(exclude_from_sim no)
+		(in_bom yes)
+		(on_board yes)
+		(dnp no)
+		(fields_autoplaced yes)
+		(property "Reference" "#PWR028"
+			(at 165.1 82.55 0)
+			(effects
+				(font
+					(size 1.27 1.27)
+				)
+				(hide yes)
+			)
+		)
+		(property "Value" "VBUS"
+			(at 165.1 73.66 0)
+			(effects
+				(font
+					(size 1.27 1.27)
+				)
+			)
+		)
+		(property "Footprint" ""
+			(at 165.1 78.74 0)
+			(effects
+				(font
+					(size 1.27 1.27)
+				)
+				(hide yes)
+			)
+		)
+		(property "Datasheet" ""
+			(at 165.1 78.74 0)
+			(effects
+				(font
+					(size 1.27 1.27)
+				)
+				(hide yes)
+			)
+		)
+		(property "Description" "Power symbol creates a global label with name \"VBUS\""
+			(at 165.1 78.74 0)
+			(effects
+				(font
+					(size 1.27 1.27)
+				)
+				(hide yes)
+			)
+		)
+		(pin "1"
+		)
+		(instances
+			(project "skibidi-usb-c-hub"
+				(path "/ba8238db-cbbe-49a0-8684-36588779fc6b/6f59b006-c39b-4f95-9bd5-f3ad5c9f2e1d"
+					(reference "#PWR031")
+					(unit 1)
+				)
+				(path "/ba8238db-cbbe-49a0-8684-36588779fc6b/a20e208f-9c1f-498b-b7e6-c187e8f066dd"
+					(reference "#PWR028")
+					(unit 1)
+				)
+				(path "/ba8238db-cbbe-49a0-8684-36588779fc6b/a3f216c1-5ccc-45d3-8b9e-12c0f2e53f02"
+					(reference "#PWR029")
+					(unit 1)
+				)
+				(path "/ba8238db-cbbe-49a0-8684-36588779fc6b/fb8800a7-8efe-42d7-a8d1-e327d54fdf66"
+					(reference "#PWR030")
+					(unit 1)
+				)
